Commit message: Migrate simulation from Gazebo Classic to Gazebo Jetty
- URDF: gz rgbd_camera, gpu_lidar and imu sensors, gz_ros2_control
- gui_launch: ros_gz_sim world + create, ros_gz_bridge config
- Replace the Classic-only Livox plugin with gpu_lidar plus a new
  pointcloud_to_livox node that republishes Livox CustomMsg
- diff_drive_controller takes TwistStamped: topic_remapper stamps
  /cmd_vel; Nav2 keeps unstamped /cmd_vel

Co-Authored-By: Claude Opus 5.5 <noreply@anthropic.com>

File: lunabot_description/urdf/v1_bot.urdf.xacro (robot description, xacro)
@@ -294,5 +294,4 @@
     </gazebo>
     <gazebo reference="front_right_wheel_link">
-      <material>Gazebo/Grey</material>
       <mu>1.0</mu>
       <mu2>1.0</mu2>
@@ -309,5 +308,4 @@
     </gazebo>
     <gazebo reference="front_left_wheel_link">
-      <material>Gazebo/Grey</material>
       <mu>1.0</mu>
       <mu2>1.0</mu2>
@@ -324,5 +322,4 @@
     </gazebo>
     <gazebo reference="rear_right_wheel_link">
-      <material>Gazebo/Grey</material>
       <mu>1.0</mu>
       <mu2>1.0</mu2>
@@ -339,5 +336,4 @@
     </gazebo>
     <gazebo reference="rear_left_wheel_link">
-      <material>Gazebo/Grey</material>
       <mu>1.0</mu>
       <mu2>1.0</mu2>
@@ -354,5 +350,5 @@
     </gazebo>
     <gazebo reference="camera_front_link">
-      <sensor type="depth" name="camera_front">
+      <sensor type="rgbd_camera" name="camera_front">
         <pose>0 0 0 0 0 0</pose>
         <update_rate>60.0</update_rate>
@@ -377,20 +373,10 @@
           </clip>
         </camera>
-        <plugin name="camera_front_controller" filename="libgazebo_ros_camera.so">
-          <ros>
-            <remapping>/camera_front/image_raw:=/camera_front/color/image_raw</remapping>
-            <remapping>/camera_front/points:=/camera_front/color/points</remapping>
-            <remapping>/camera_front/camera_info:=/camera_front/color/camera_info</remapping>
-            <remapping>/camera_front/depth/image_raw:=/camera_front/depth/image_rect_raw</remapping>
-          </ros>
-          <frame_name>camera_front_optical_link</frame_name>
-          <publish_tf>false</publish_tf>
-          <publish_point_cloud>true</publish_point_cloud>
-        </plugin>
+        <topic>camera_front</topic>
+        <gz_frame_id>camera_front_optical_link</gz_frame_id>
       </sensor>
-      <material>Gazebo/Grey</material>
     </gazebo>
     <gazebo reference="camera_back_link">
-      <sensor type="depth" name="camera_back">
+      <sensor type="rgbd_camera" name="camera_back">
         <pose>0 0 0 0 0 0</pose>
         <update_rate>60.0</update_rate>
@@ -415,20 +401,10 @@
           </clip>
         </camera>
-        <plugin name="camera_back_controller" filename="libgazebo_ros_camera.so">
-          <ros>
-            <remapping>/camera_back/image_raw:=/camera_back/color/image_raw</remapping>
-            <remapping>/camera_back/points:=/camera_back/color/points</remapping>
-            <remapping>/camera_back/camera_info:=/camera_back/color/camera_info</remapping>
-            <remapping>/camera_back/depth/image_raw:=/camera_back/depth/image_rect_raw</remapping>
-          </ros>
-          <frame_name>camera_back_optical_link</frame_name>
-          <publish_tf>false</publish_tf>
-          <publish_point_cloud>true</publish_point_cloud>
-        </plugin>
+        <topic>camera_back</topic>
+        <gz_frame_id>camera_back_optical_link</gz_frame_id>
       </sensor>
-      <material>Gazebo/Grey</material>
     </gazebo>
     <gazebo reference="camera_fisheye_link">
-      <sensor type="depth" name="camera_fisheye">
+      <sensor type="rgbd_camera" name="camera_fisheye">
         <pose>0 0 0 0 0 0</pose>
         <update_rate>60.0</update_rate>
@@ -453,57 +429,44 @@
           </clip>
         </camera>
-        <plugin name="camera_fisheye_controller" filename="libgazebo_ros_camera.so">
-          <ros>
-            <remapping>/camera_fisheye/image_raw:=/camera_fisheye/color/image_raw</remapping>
-            <remapping>/camera_fisheye/points:=/camera_fisheye/color/points</remapping>
-            <remapping>/camera_fisheye/camera_info:=/camera_fisheye/color/camera_info</remapping>
-            <remapping>/camera_fisheye/depth/image_raw:=/camera_fisheye/depth/image_rect_raw</remapping>
-          </ros>
-          <frame_name>camera_fisheye_optical_link</frame_name>
-          <publish_tf>false</publish_tf>
-          <publish_point_cloud>true</publish_point_cloud>
-        </plugin>
+        <topic>camera_fisheye</topic>
+        <gz_frame_id>camera_fisheye_optical_link</gz_frame_id>
       </sensor>
-      <material>Gazebo/Grey</material>
     </gazebo>
     <gazebo reference="livox_frame">
-      <sensor type="ray" name="mid360_lidar_sensor">
+      <sensor type="gpu_lidar" name="mid360_lidar_sensor">
+        <!-- Replaces the Gazebo Classic Livox plugin; lunabot_util/pointcloud_to_livox turns the
+             bridged PointCloud2 into the CustomMsg on /livox/lidar that the real driver publishes -->
         <always_on>true</always_on>
         <pose>0 0 0 0 0 0</pose>
         <visualize>false</visualize>
         <update_rate>10</update_rate>
-        <plugin name="mid360_plugin" filename="libros2_livox.so">
-          <ray>
-            <scan>
-              <horizontal>
-                <samples>100</samples>
-                <resolution>1</resolution>
-                <min_angle>0</min_angle>
-                <max_angle>6.2831852</max_angle>
-              </horizontal>
-              <vertical>
-                <samples>360</samples>
-                <resolution>1</resolution>
-                <min_angle>-0.126</min_angle>
-                <max_angle>0.964</max_angle>
-              </vertical>
-            </scan>
-            <range>
-              <min>0.1</min>
-              <max>50.0</max>
-              <resolution>0.002</resolution>
-            </range>
-            <noise>
-              <type>gaussian</type>
-              <mean>0.0</mean>
-              <stddev>0.01</stddev>
-            </noise>
-          </ray>
-          <visualize>false</visualize>
-          <samples>20000</samples>
-          <downsample>2</downsample>
-          <csv_file_name>$(find ros2_livox_simulation)/scan_mode/mid360.csv</csv_file_name>
-          <topic>livox/lidar</topic>
-        </plugin>
+        <topic>livox/lidar_points</topic>
+        <gz_frame_id>livox_frame</gz_frame_id>
+        <lidar>
+          <scan>
+            <horizontal>
+              <samples>360</samples>
+              <resolution>1</resolution>
+              <min_angle>-3.1415926</min_angle>
+              <max_angle>3.1415926</max_angle>
+            </horizontal>
+            <vertical>
+              <samples>32</samples>
+              <resolution>1</resolution>
+              <min_angle>-0.126</min_angle>
+              <max_angle>0.964</max_angle>
+            </vertical>
+          </scan>
+          <range>
+            <min>0.1</min>
+            <max>50.0</max>
+            <resolution>0.002</resolution>
+          </range>
+          <noise>
+            <type>gaussian</type>
+            <mean>0.0</mean>
+            <stddev>0.01</stddev>
+          </noise>
+        </lidar>
       </sensor>
     </gazebo>
@@ -514,30 +477,29 @@
         <update_rate>100</update_rate>
         <visualize>true</visualize>
-        <plugin filename="libgazebo_ros_imu_sensor.so" name="imu_plugin">
-          <ros>
-            <namespace></namespace>
-            <remapping>~/out:=/livox/imu</remapping>
-          </ros>
-          <bodyName>mid360_imu_link</bodyName>
-          <gaussianNoise>0.01</gaussianNoise>
-          <xyzOffset>0 0 0</xyzOffset>
-          <rpyOffset>0 0 0</rpyOffset>
-          <frameName>mid360_imu_link</frameName>
-          <publish_tf>false</publish_tf>
-          <initialOrientationAsReference>false</initialOrientationAsReference>
-        </plugin>
+        <topic>livox/imu</topic>
+        <gz_frame_id>mid360_imu_link</gz_frame_id>
+        <imu>
+          <angular_velocity>
+            <x><noise type="gaussian"><mean>0.0</mean><stddev>0.01</stddev></noise></x>
+            <y><noise type="gaussian"><mean>0.0</mean><stddev>0.01</stddev></noise></y>
+            <z><noise type="gaussian"><mean>0.0</mean><stddev>0.01</stddev></noise></z>
+          </angular_velocity>
+          <linear_acceleration>
+            <x><noise type="gaussian"><mean>0.0</mean><stddev>0.01</stddev></noise></x>
+            <y><noise type="gaussian"><mean>0.0</mean><stddev>0.01</stddev></noise></y>
+            <z><noise type="gaussian"><mean>0.0</mean><stddev>0.01</stddev></noise></z>
+          </linear_acceleration>
+        </imu>
         <pose>0 0 0 0 0 0</pose>
       </sensor>
     </gazebo>
     <gazebo>
-      <plugin name="gazebo_ros2_control" filename="libgazebo_ros2_control.so">
-        <robot_param>robot_description</robot_param>
-        <robot_param_node>robot_state_publisher</robot_param_node>
+      <plugin filename="gz_ros2_control-system" name="gz_ros2_control::GazeboSimROS2ControlPlugin">
         <parameters>$(find lunabot_config)/params/gazebo/gazebo_v1_bot_params.yaml</parameters>
       </plugin>
     </gazebo>
-    <ros2_control name="GazeboSystem" type="system">
+    <ros2_control name="GazeboSimSystem" type="system">
       <hardware>
-        <plugin>gazebo_ros2_control/GazeboSystem</plugin>
+        <plugin>gz_ros2_control/GazeboSimSystem</plugin>
       </hardware>
       <joint name="base_front_right_wheel_joint">

File: lunabot_description/urdf/v2_bot.urdf.xacro (robot description, xacro)
@@ -336,5 +336,4 @@
     </gazebo>
     <gazebo reference="front_right_wheel_link">
-      <material>Gazebo/Grey</material>
       <mu>1.0</mu>
       <mu2>1.0</mu2>
@@ -351,5 +350,4 @@
     </gazebo>
     <gazebo reference="front_left_wheel_link">
-      <material>Gazebo/Grey</material>
       <mu>1.0</mu>
       <mu2>1.0</mu2>
@@ -366,5 +364,4 @@
     </gazebo>
     <gazebo reference="rear_right_wheel_link">
-      <material>Gazebo/Grey</material>
       <mu>1.0</mu>
       <mu2>1.0</mu2>
@@ -381,5 +378,4 @@
     </gazebo>
     <gazebo reference="rear_left_wheel_link">
-      <material>Gazebo/Grey</material>
       <mu>1.0</mu>
       <mu2>1.0</mu2>
@@ -396,5 +392,5 @@
     </gazebo>
     <gazebo reference="camera_front_link">
-      <sensor type="depth" name="camera_front">
+      <sensor type="rgbd_camera" name="camera_front">
         <pose>0 0 0 0 0 0</pose>
         <update_rate>60.0</update_rate>
@@ -419,20 +415,10 @@
           </clip>
         </camera>
-        <plugin name="camera_front_controller" filename="libgazebo_ros_camera.so">
-          <ros>
-            <remapping>/camera_front/image_raw:=/camera_front/color/image_raw</remapping>
-            <remapping>/camera_front/points:=/camera_front/color/points</remapping>
-            <remapping>/camera_front/camera_info:=/camera_front/color/camera_info</remapping>
-            <remapping>/camera_front/depth/image_raw:=/camera_front/depth/image_rect_raw</remapping>
-          </ros>
-          <frame_name>camera_front_optical_link</frame_name>
-          <publish_tf>false</publish_tf>
-          <publish_point_cloud>true</publish_point_cloud>
-        </plugin>
+        <topic>camera_front</topic>
+        <gz_frame_id>camera_front_optical_link</gz_frame_id>
       </sensor>
-      <material>Gazebo/Grey</material>
     </gazebo>
     <gazebo reference="camera_back_link">
-      <sensor type="depth" name="camera_back">
+      <sensor type="rgbd_camera" name="camera_back">
         <pose>0 0 0 0 0 0</pose>
         <update_rate>60.0</update_rate>
@@ -457,20 +443,10 @@
           </clip>
         </camera>
-        <plugin name="camera_back_controller" filename="libgazebo_ros_camera.so">
-          <ros>
-            <remapping>/camera_back/image_raw:=/camera_back/color/image_raw</remapping>
-            <remapping>/camera_back/points:=/camera_back/color/points</remapping>
-            <remapping>/camera_back/camera_info:=/camera_back/color/camera_info</remapping>
-            <remapping>/camera_back/depth/image_raw:=/camera_back/depth/image_rect_raw</remapping>
-          </ros>
-          <frame_name>camera_back_optical_link</frame_name>
-          <publish_tf>false</publish_tf>
-          <publish_point_cloud>true</publish_point_cloud>
-        </plugin>
+        <topic>camera_back</topic>
+        <gz_frame_id>camera_back_optical_link</gz_frame_id>
       </sensor>
-      <material>Gazebo/Grey</material>
     </gazebo>
     <gazebo reference="camera_fisheye_link">
-      <sensor type="depth" name="camera_fisheye">
+      <sensor type="rgbd_camera" name="camera_fisheye">
         <pose>0 0 0 0 0 0</pose>
         <update_rate>60.0</update_rate>
@@ -495,57 +471,44 @@
           </clip>
         </camera>
-        <plugin name="camera_fisheye_controller" filename="libgazebo_ros_camera.so">
-          <ros>
-            <remapping>/camera_fisheye/image_raw:=/camera_fisheye/color/image_raw</remapping>
-            <remapping>/camera_fisheye/points:=/camera_fisheye/color/points</remapping>
-            <remapping>/camera_fisheye/camera_info:=/camera_fisheye/color/camera_info</remapping>
-            <remapping>/camera_fisheye/depth/image_raw:=/camera_fisheye/depth/image_rect_raw</remapping>
-          </ros>
-          <frame_name>camera_fisheye_optical_link</frame_name>
-          <publish_tf>false</publish_tf>
-          <publish_point_cloud>true</publish_point_cloud>
-        </plugin>
+        <topic>camera_fisheye</topic>
+        <gz_frame_id>camera_fisheye_optical_link</gz_frame_id>
       </sensor>
-      <material>Gazebo/Grey</material>
     </gazebo>
     <gazebo reference="livox_frame">
-      <sensor type="ray" name="mid360_lidar_sensor">
+      <sensor type="gpu_lidar" name="mid360_lidar_sensor">
+        <!-- Replaces the Gazebo Classic Livox plugin; lunabot_util/pointcloud_to_livox turns the
+             bridged PointCloud2 into the CustomMsg on /livox/lidar that the real driver publishes -->
         <always_on>true</always_on>
         <pose>0 0 0 0 0 0</pose>
         <visualize>false</visualize>
         <update_rate>10</update_rate>
-        <plugin name="mid360_plugin" filename="libros2_livox.so">
-          <ray>
-            <scan>
-              <horizontal>
-                <samples>100</samples>
-                <resolution>1</resolution>
-                <min_angle>0</min_angle>
-                <max_angle>6.2831852</max_angle>
-              </horizontal>
-              <vertical>
-                <samples>360</samples>
-                <resolution>1</resolution>
-                <min_angle>-0.126</min_angle>
-                <max_angle>0.964</max_angle>
-              </vertical>
-            </scan>
-            <range>
-              <min>0.1</min>
-              <max>50.0</max>
-              <resolution>0.002</resolution>
-            </range>
-            <noise>
-              <type>gaussian</type>
-              <mean>0.0</mean>
-              <stddev>0.01</stddev>
-            </noise>
-          </ray>
-          <visualize>false</visualize>
-          <samples>20000</samples>
-          <downsample>2</downsample>
-          <csv_file_name>$(find ros2_livox_simulation)/scan_mode/mid360.csv</csv_file_name>
-          <topic>livox/lidar</topic>
-        </plugin>
+        <topic>livox/lidar_points</topic>
+        <gz_frame_id>livox_frame</gz_frame_id>
+        <lidar>
+          <scan>
+            <horizontal>
+              <samples>360</samples>
+              <resolution>1</resolution>
+              <min_angle>-3.1415926</min_angle>
+              <max_angle>3.1415926</max_angle>
+            </horizontal>
+            <vertical>
+              <samples>32</samples>
+              <resolution>1</resolution>
+              <min_angle>-0.126</min_angle>
+              <max_angle>0.964</max_angle>
+            </vertical>
+          </scan>
+          <range>
+            <min>0.1</min>
+            <max>50.0</max>
+            <resolution>0.002</resolution>
+          </range>
+          <noise>
+            <type>gaussian</type>
+            <mean>0.0</mean>
+            <stddev>0.01</stddev>
+          </noise>
+        </lidar>
       </sensor>
     </gazebo>
@@ -556,30 +519,29 @@
         <update_rate>100</update_rate>
         <visualize>true</visualize>
-        <plugin filename="libgazebo_ros_imu_sensor.so" name="imu_plugin">
-          <ros>
-            <namespace></namespace>
-            <remapping>~/out:=/livox/imu</remapping>
-          </ros>
-          <bodyName>mid360_imu_link</bodyName>
-          <gaussianNoise>0.01</gaussianNoise>
-          <xyzOffset>0 0 0</xyzOffset>
-          <rpyOffset>0 0 0</rpyOffset>
-          <frameName>mid360_imu_link</frameName>
-          <publish_tf>false</publish_tf>
-          <initialOrientationAsReference>false</initialOrientationAsReference>
-        </plugin>
+        <topic>livox/imu</topic>
+        <gz_frame_id>mid360_imu_link</gz_frame_id>
+        <imu>
+          <angular_velocity>
+            <x><noise type="gaussian"><mean>0.0</mean><stddev>0.01</stddev></noise></x>
+            <y><noise type="gaussian"><mean>0.0</mean><stddev>0.01</stddev></noise></y>
+            <z><noise type="gaussian"><mean>0.0</mean><stddev>0.01</stddev></noise></z>
+          </angular_velocity>
+          <linear_acceleration>
+            <x><noise type="gaussian"><mean>0.0</mean><stddev>0.01</stddev></noise></x>
+            <y><noise type="gaussian"><mean>0.0</mean><stddev>0.01</stddev></noise></y>
+            <z><noise type="gaussian"><mean>0.0</mean><stddev>0.01</stddev></noise></z>
+          </linear_acceleration>
+        </imu>
         <pose>0 0 0 0 0 0</pose>
       </sensor>
     </gazebo>
     <gazebo>
-      <plugin name="gazebo_ros2_control" filename="libgazebo_ros2_control.so">
-        <robot_param>robot_description</robot_param>
-        <robot_param_node>robot_state_publisher</robot_param_node>
+      <plugin filename="gz_ros2_control-system" name="gz_ros2_control::GazeboSimROS2ControlPlugin">
         <parameters>$(find lunabot_config)/params/gazebo/gazebo_v2_bot_params.yaml</parameters>
       </plugin>
     </gazebo>
-    <ros2_control name="GazeboSystem" type="system">
+    <ros2_control name="GazeboSimSystem" type="system">
       <hardware>
-        <plugin>gazebo_ros2_control/GazeboSystem</plugin>
+        <plugin>gz_ros2_control/GazeboSimSystem</plugin>
       </hardware>
       <joint name="base_front_right_wheel_joint">
